File: Project 1 LED Torch/Project 1 LED Torch.kicad_sch (KiCad schematic)
At the start: 0 parts

Commit message: Schematic design
Parts:
- added BT1: Battery_Cell, Battery:BatteryHolder_Keystone_1058_1x2032, symbol Device:Battery_Cell
- added D1: LED, LED_THT:LED_D5.0mm, symbol Device:LED
- added R1: R, Resistor_THT:R_Axial_DIN0204_L3.6mm_D1.6mm_P7.62mm_Horizontal, symbol Device:R
- added SW1: SW_DPDT_x2, Button_Switch_THT:SW_TH_Tactile_Omron_B3F-100x, symbol Switch:SW_DPST_x2
Connections:
- new net: R1.2, SW1.1 (A)
- new net LED_anode: D1.2 (A), R1.1
- new net LED_cathode: BT1.2 (-), D1.1 (K)
- new net bat_pos: BT1.1 (+), SW1.2 (B)
Other:
- note added: "LED Torch"
